Commit message: update mimic joint tutorial for newer joint_trajectory_controller with mimic joint support

File: urdf/mimic_joint_gazebo_tutorial.urdf.xacro (robot description, xacro)
@@ -26,22 +26,4 @@
     </material>
   </xacro:property>
-  <xacro:macro name="mimic_joint_plugin_gazebo" params="name_prefix parent_joint mimic_joint has_pid:=false multiplier:=1.0 offset:=0 sensitiveness:=0.0 max_effort:=1.0 robot_namespace:=''">
-    <gazebo>
-      <plugin name="${name_prefix}mimic_joint_plugin" filename="libroboticsgroup_gazebo_mimic_joint_plugin.so">
-        <joint>${parent_joint}</joint>
-        <mimicJoint>${mimic_joint}</mimicJoint>
-        <xacro:if value="${has_pid}">                     <!-- if set to true, PID parameters from "/gazebo_ros_control/pid_gains/${mimic_joint}" are loaded -->
-          <hasPID />
-        </xacro:if>
-        <multiplier>${multiplier}</multiplier>
-        <offset>${offset}</offset>
-        <sensitiveness>${sensitiveness}</sensitiveness>   <!-- if absolute difference between setpoint and process value is below this threshold, do nothing; 0.0 = disable [rad] -->
-        <maxEffort>${max_effort}</maxEffort>              <!-- only taken into account if has_pid:=true [Nm] -->
-        <xacro:unless value="${robot_namespace == ''}">
-          <robotNamespace>($robot_namespace)</robotNamespace>
-        </xacro:unless>
-      </plugin>
-    </gazebo>
-  </xacro:macro>
   <xacro:macro name="controller_plugin_gazebo" params="robot_namespace:=''">
     <gazebo>
@@ -129,10 +111,7 @@
     <axis xyz="1 0 0" />
     <limit lower="0" upper="${pi / 2}" velocity="0.7" effort="1000" />
-    <mimic joint="right_finger_joint" multiplier="1" offset="0" />
+    <mimic joint="right_finger_joint" multiplier="0.5" offset="0" />
     <dynamics damping="0.02" friction="0.0" />
   </joint>
-  <xacro:mimic_joint_plugin_gazebo name_prefix="left_finger_joint"
-    parent_joint="right_finger_joint" mimic_joint="left_finger_joint"
-    has_pid="true" multiplier="1.0" max_effort="10.0" />
   <link name="left_finger">
     <visual>
@@ -156,8 +135,4 @@
     <material>Gazebo/Red</material>
   </gazebo>
-  <!-- DO NOT add a transmission for the left finger joint. We want the left
-       finger joint to be controlled by the mimic plugin. If we add a
-       transmission, the ros_control plugin will try to control this joint. -->
-  <!--
   <transmission name="left_finger_joint_trans">
     <type>transmission_interface/SimpleTransmission</type>
@@ -169,4 +144,3 @@
     </actuator>
   </transmission>
-  -->
 </robot>
